File: PCB/PCB.kicad_pcb (KiCad board)
At the start: 4 copper layers, 96 x 60 mm, 72 parts, among them J1 USB_C_Receptacle_USB2.0_16P, J2 Conn_01x04_Pin, J3 Conn_01x12_Pin, J4 Conn_01x12_Pin, J5 Power select, SW1 SW_Push, U1 STM32L052C8Tx, U2 SX1262IMLTRT, U3 USBLC6-2P6, U4 AP2112K-3.3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

Commit message: PCB MOSTLY DONE
Parts:
- removed J3, J4: Conn_01x12_Pin, Connector_PinHeader_2.54mm:PinHeader_1x12_P2.54mm_Vertical
- added C26: 12pF, Capacitor_SMD:C_0402_1005Metric, F.Cu at (199.5, 82.0)
- added C27: 12pF, Capacitor_SMD:C_0402_1005Metric, F.Cu at (196.2, 84.8)
- added TP3: TestPoint, TestPoint:TestPoint_Pad_D1.0mm, F.Cu at (215.8, 78.2)
- added TP4: TestPoint, TestPoint:TestPoint_Pad_D1.0mm, B.Cu at (185.0, 91.8)
- added TP5: TestPoint, TestPoint:TestPoint_Pad_D1.0mm, B.Cu at (190.8, 89.0)
- added TP6: TestPoint, TestPoint:TestPoint_Pad_D1.0mm, B.Cu at (185.0, 94.0)
- AE1: value Antenna -> Antenna_Shield; footprint Connector_PinHeader_2.54mm:PinHeader_1x01_P2.54mm_Vertical -> Connector_Coaxial:SMA_Amphenol_901-144_Vertical
- C10, C5, C6, C8: value 10uF -> 4.7uF
- Y1: value Crystal_GND24 -> 32Mhz
- moved AE1 5.70 mm to (215.5, 84.7)
- moved G*** 4.37 mm to (169.5, 87.8)
- moved C17 2.20 mm to (195.5, 88.5)
- moved C18 2.20 mm to (195.0, 90.8)
- moved C20 2.20 mm to (202.5, 85.8)
- moved C21 2.20 mm to (202.5, 86.8)
- moved C22 2.20 mm to (208.9, 89.8)
- moved L2 2.20 mm to (194.5, 89.2)
- moved L3 2.20 mm to (202.0, 88.3)
- moved U2 2.20 mm to (198.7, 90.0)
- moved Y1 2.20 mm to (198.9, 84.4)
- moved C19 2.20 mm to (200.5, 86.8)
- moved C23 2.20 mm to (210.4, 90.3)
- moved C24 2.20 mm to (213.3, 90.3)
- moved C25 2.20 mm to (206.5, 91.5)
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Connections:
- net +BATT renamed +BATT_3P7
Routing:
- net /TS: track 0.00 -> 23.0 mm, vias 0 -> 2
- net GND: track 53.8 -> 71.0 mm, vias 167 -> 159
- net Net-(AE1-A): track 3.42 -> 7.27 mm
- net /MOSI: track 45.4 -> 49.0 mm, vias 4 -> 5
- net /SX_NRST: track 38.3 -> 35.6 mm
- net /SX_NSS: track 42.1 -> 39.4 mm
- net /CLK: track 49.1 -> 51.4 mm
- net /SX_BUSY: track 30.7 -> 28.6 mm
- net /SX_DIO1: track 25.6 -> 23.7 mm
- net /SX_XTB: track 3.05 -> 4.65 mm
- net /SX_XTA: track 4.96 -> 6.53 mm
- net Net-(U5-~{VSET}): track 0.00 -> 1.30 mm
- net VBUS: track 17.2 -> 16.0 mm
- net /SCK: track 106.8 -> 107.6 mm, vias 2 -> 3
- net +3V3: track 50.1 -> 50.8 mm
