File: PCB/PCB.kicad_sch (KiCad schematic)
At the start: 71 parts, among them J1 USB_C_Receptacle_USB2.0_16P, J2 Conn_01x04_Pin, J3 Conn_01x12_Pin, J4 Conn_01x12_Pin, J5 Power select, SW1 SW_Push, U1 STM32L052C8Tx, U2 SX1262IMLTRT, U3 USBLC6-2P6, U4 AP2112K-3.3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

Commit message: PCB MOSTLY DONE
Parts:
- removed AE1: Antenna, Connector_PinHeader_2.54mm:PinHeader_1x01_P2.54mm_Vertical, symbol Device:Antenna
- removed J3, J4: Conn_01x12_Pin, Connector_PinHeader_2.54mm:PinHeader_1x12_P2.54mm_Vertical, symbol Connector:Conn_01x12_Pin
- added AE1: Antenna_Shield, Connector_Coaxial:SMA_Amphenol_901-144_Vertical, symbol Device:Antenna_Shield
- added C26, C27: 12pF, Capacitor_SMD:C_0402_1005Metric, symbol Device:C
- added TP3, TP4, TP5, TP6: TestPoint, TestPoint:TestPoint_Pad_D1.0mm, symbol Connector:TestPoint
- Y1: value Crystal_GND24 -> 32Mhz
Connections:
- net CLK: now also TP6.1
- net GND: now also AE1.2 (Shield), C26.1, C27.1, TP3.1
- net MISO: now also TP5.1
- net MOSI: now also TP4.1
- net SX_XTA: now also C26.2
- net SX_XTB: now also C27.2
- net at C24.1, L4.2: now also AE1.1 (A)
- net +BATT renamed +BATT_3P7
Other:
- moved on the sheet: Y1
